Commit message: Changes made by satyanshu

File: nextup_moveit_config/config/robot_nextup.ros2_control.xacro (robot description, xacro)
@@ -1,5 +1,5 @@
 <?xml version="1.0"?>
 <robot xmlns:xacro="http://www.ros.org/wiki/xacro">
-  <xacro:macro name="robot_nextup_ros2_control" params="initial_positions_file vendor:=innovance product:=robot1">
+  <xacro:macro name="robot_nextup_ros2_control" params="initial_positions_file vendor:=innovance product:=cobot">
     <xacro:property name="initial_positions" value="${xacro.load_yaml(initial_positions_file)['initial_positions']}"/>
     <xacro:property name="slave_config_dir" value="$(find nextup_moveit_config)/config/${vendor}/${product}"/>

File: nextup_moveit_config/config/robot_nextup.urdf.xacro (robot description, xacro)
@@ -2,5 +2,5 @@
 <robot xmlns:xacro="http://www.ros.org/wiki/xacro" name="robot_nextup">
     <!-- SELECT ROBOT HERE -->
-    <xacro:property name="robot_type" value="robot1"/>
+    <xacro:property name="robot_type" value="cobot"/>
     <xacro:arg name="initial_positions_file" default="initial_positions.yaml" />
     <xacro:if value="${robot_type == 'robot'}">

Commit message: change made to joint_limits.yaml kinematics.yaml

File: nextup_moveit_config/config/robot_nextup.ros2_control.xacro (robot description, xacro)
@@ -1,5 +1,5 @@
 <?xml version="1.0"?>
 <robot xmlns:xacro="http://www.ros.org/wiki/xacro">
-  <xacro:macro name="robot_nextup_ros2_control" params="initial_positions_file vendor:=innovance product:=cobot">
+  <xacro:macro name="robot_nextup_ros2_control" params="initial_positions_file vendor:=innovance product:=robot1">
     <xacro:property name="initial_positions" value="${xacro.load_yaml(initial_positions_file)['initial_positions']}"/>
     <xacro:property name="slave_config_dir" value="$(find nextup_moveit_config)/config/${vendor}/${product}"/>

File: nextup_moveit_config/config/robot_nextup.urdf.xacro (robot description, xacro)
@@ -2,5 +2,5 @@
 <robot xmlns:xacro="http://www.ros.org/wiki/xacro" name="robot_nextup">
     <!-- SELECT ROBOT HERE -->
-    <xacro:property name="robot_type" value="cobot"/>
+    <xacro:property name="robot_type" value="robot1"/>
     <xacro:arg name="initial_positions_file" default="initial_positions.yaml" />
     <xacro:if value="${robot_type == 'robot'}">

Commit message: latest_software_stack

File: nextup_moveit_config/config/robot_nextup.ros2_control.xacro (robot description, xacro)
@@ -1,5 +1,5 @@
 <?xml version="1.0"?>
 <robot xmlns:xacro="http://www.ros.org/wiki/xacro">
-  <xacro:macro name="robot_nextup_ros2_control" params="initial_positions_file vendor:=innovance product:=robot1">
+  <xacro:macro name="robot_nextup_ros2_control" params="initial_positions_file vendor:=innovance product:=cobot">
     <xacro:property name="initial_positions" value="${xacro.load_yaml(initial_positions_file)['initial_positions']}"/>
     <xacro:property name="slave_config_dir" value="$(find nextup_moveit_config)/config/${vendor}/${product}"/>
@@ -26,8 +26,10 @@
         <command_interface name="dos"/>
         <command_interface name="emergency_trigger"/>
+        <command_interface name="runway_protection"/>
+        <command_interface name="max_torque"/>
         <ec_module name="ZeroErr">
           <plugin>ethercat_generic_plugins/EcCiA402Drive</plugin>
           <param name="alias">0</param>
-          <param name="position">0</param>
+          <param name="position">6</param>
           <param name="mode_of_operation">9</param>
           <param name="slave_config">${slave_config_dir}/joint1.yaml</param>
@@ -50,4 +52,6 @@
         <command_interface name="dos"/>
         <command_interface name="emergency_trigger"/>
+        <command_interface name="runway_protection"/>
+        <command_interface name="max_torque"/>
         <ec_module name="ZeroErr">
           <plugin>ethercat_generic_plugins/EcCiA402Drive</plugin>
@@ -74,4 +78,6 @@
         <command_interface name="dos"/>
         <command_interface name="emergency_trigger"/>
+        <command_interface name="runway_protection"/>
+        <command_interface name="max_torque"/>
         <ec_module name="ZeroErr">
           <plugin>ethercat_generic_plugins/EcCiA402Drive</plugin>
@@ -98,4 +104,6 @@
         <command_interface name="dos"/>
         <command_interface name="emergency_trigger"/>
+        <command_interface name="runway_protection"/>
+        <command_interface name="max_torque"/>
         <ec_module name="ZeroErr">
           <plugin>ethercat_generic_plugins/EcCiA402Drive</plugin>
@@ -122,4 +130,6 @@
         <command_interface name="dos"/>
         <command_interface name="emergency_trigger"/>
+        <command_interface name="runway_protection"/>
+        <command_interface name="max_torque"/>
         <ec_module name="ZeroErr">
           <plugin>ethercat_generic_plugins/EcCiA402Drive</plugin>
@@ -146,4 +156,6 @@
         <command_interface name="dos"/>
         <command_interface name="emergency_trigger"/>
+        <command_interface name="runway_protection"/>
+        <command_interface name="max_torque"/>
         <ec_module name="ZeroErr">
           <plugin>ethercat_generic_plugins/EcCiA402Drive</plugin>
@@ -154,4 +166,15 @@
         </ec_module>
       </joint>
+      <gpio name="gpio1">
+        <command_interface name="d_output_allbit"/>
+        <state_interface name="d_input_allbit"/>
+        <state_interface name="error_code"/>
+        <ec_module name="RTU">
+          <plugin>ethercat_generic_plugins/GenericEcSlave</plugin>
+          <param name="alias">0</param>
+          <param name="position">0</param>
+          <param name="slave_config">/home/nextup/NextupRobot/src/nextup_moveit_config/config/innovance/do_di.yaml</param>
+        </ec_module>
+      </gpio>
     </ros2_control>
 </xacro:macro>

File: nextup_moveit_config/config/robot_nextup.urdf.xacro (robot description, xacro)
@@ -2,5 +2,5 @@
 <robot xmlns:xacro="http://www.ros.org/wiki/xacro" name="robot_nextup">
     <!-- SELECT ROBOT HERE -->
-    <xacro:property name="robot_type" value="robot1"/>
+    <xacro:property name="robot_type" value="cobot"/>
     <xacro:arg name="initial_positions_file" default="initial_positions.yaml" />
     <xacro:if value="${robot_type == 'robot'}">

Commit message: GSC_SBN_19_20_ROBOT1

File: nextup_moveit_config/config/robot_nextup.ros2_control.xacro (robot description, xacro)
@@ -1,5 +1,5 @@
 <?xml version="1.0"?>
 <robot xmlns:xacro="http://www.ros.org/wiki/xacro">
-  <xacro:macro name="robot_nextup_ros2_control" params="initial_positions_file vendor:=innovance product:=cobot">
+  <xacro:macro name="robot_nextup_ros2_control" params="initial_positions_file vendor:=innovance product:=robot1">
     <xacro:property name="initial_positions" value="${xacro.load_yaml(initial_positions_file)['initial_positions']}"/>
     <xacro:property name="slave_config_dir" value="$(find nextup_moveit_config)/config/${vendor}/${product}"/>
@@ -8,5 +8,5 @@
         <plugin>ethercat_driver/EthercatDriver</plugin>
         <param name="master_id">0</param>
-        <param name="control_frequency">200</param>
+        <param name="control_frequency">125</param>
       </hardware>
       <joint name="joint1">

File: nextup_moveit_config/config/robot_nextup.urdf.xacro (robot description, xacro)
@@ -2,5 +2,5 @@
 <robot xmlns:xacro="http://www.ros.org/wiki/xacro" name="robot_nextup">
     <!-- SELECT ROBOT HERE -->
-    <xacro:property name="robot_type" value="cobot"/>
+    <xacro:property name="robot_type" value="robot1"/>
     <xacro:arg name="initial_positions_file" default="initial_positions.yaml" />
     <xacro:if value="${robot_type == 'robot'}">

File: nextup_moveit_config/urdf/nextupRobot1.urdf copy.xacro (robot description, xacro)
@@ -67,5 +67,5 @@
             <origin
                 xyz="0.18631 1.6653E-15 0.14306"
-                rpy="0 0 0" />
+                rpy="0 0 -1.57" />
             <mass
                 value="21.096" />
@@ -81,5 +81,5 @@
             <origin
                 xyz="0 0 0"
-                rpy="0 0 0" />
+                rpy="0 0 -1.57" />
             <geometry>
                 <mesh
@@ -95,5 +95,5 @@
             <origin
                 xyz="0 0 0"
-                rpy="0 0 0" />
+                rpy="0 0 -1.57" />
             <geometry>
                 <mesh
@@ -107,5 +107,5 @@
         <origin
             xyz="0 0 0.593"
-            rpy="0 0 0" />
+            rpy="0 0 1.57" />
         <parent
             link="base_link" />
@@ -164,6 +164,6 @@
         type="revolute">
         <origin
-            xyz="0.0772577082457715 0 0.18"
-            rpy="-1.5707963267949 0.40214795034629 1.5707963267949" />
+            xyz="0.0 -0.02 0.18"
+            rpy="-1.5707963267949 -0.38324021305116 0.0" />
         <parent
             link="link1" />
@@ -223,5 +223,5 @@
         <origin
       xyz="-0.383049008063237 -0.923728021347067 0.00200000000000033"
-      rpy="3.14159265358979 0 -0.40214795034629" />
+      rpy="3.14159265358979 0 -2.5837540138" />
         <parent
             link="link2" />
@@ -281,5 +281,5 @@
         <origin
       xyz="0 0.6 0"
-      rpy="3.14159265358979 0 1.5707963267949" />
+      rpy="3.14159265358979 0 0" />
         <parent
             link="link3" />
@@ -339,5 +339,5 @@
         <origin
       xyz="0.180000001578827 0 0.105999997318973"
-      rpy="1.57079634168949 0 1.5707963267949" />
+      rpy="1.57079634168949 -1.570796326949 1.5707963267949" />
         <parent
             link="link4" />
